Commit message: add wbc

File: humanoid-legged-description/urdf/humanoid_legged_control.urdf (robot description, URDF)
Before this commit: robot humanoid_legged_description, 20 links, 19 joints
Links:
- link base_link: geometry 
- link leg_l1_link: geometry 
- link leg_l2_link: geometry 
- link leg_l3_link: geometry 
- link leg_l4_link: geometry 
- link leg_l5_link: geometry 
- link leg_l6_link: geometry 
- link leg_r1_link: geometry 
- link leg_r2_link: geometry 
- link leg_r3_link: geometry 
- link leg_r4_link: geometry 
- link leg_r5_link: geometry 
- link leg_r6_link: geometry 
