Commit message: 更换机器人模型，修复cheat controller只能转四分之一圈的Bug，调参

File: humanoid-legged-description/mjcf/humanoid_legged.urdf (robot description, URDF)
Before this commit: robot humanoid_legged_description, 14 links, 13 joints
Links:
- added link arm_l1_link, mass 0.565198; visual mesh filename=../meshes/arm_l1_link.STL
- added link arm_l2_link, mass 0.850000; visual mesh filename=../meshes/arm_l2_link.STL
- added link arm_l3_link, mass 0.700000; collision cylinder length=0.16 radius=0.04; visual mesh filename=../meshes/arm_l3_link.STL
- added link arm_l4_link, mass 0.443929; visual mesh filename=../meshes/arm_l4_link.STL
- added link arm_l5_link, mass 0.250000; collision cylinder length=0.1 radius=0.04; visual mesh filename=../meshes/arm_l5_link.STL
- added link arm_l6_link, mass 0.600000; visual mesh filename=../meshes/arm_l6_link.STL
- added link arm_r1_link, mass 0.565198; visual mesh filename=../meshes/arm_r1_link.STL
- added link arm_r2_link, mass 0.850000; visual mesh filename=../meshes/arm_r2_link.STL
- added link arm_r3_link, mass 0.700000; collision cylinder length=0.16 radius=0.04; visual mesh filename=../meshes/arm_r3_link.STL
- added link arm_r4_link, mass 0.443929; visual mesh filename=../meshes/arm_r4_link.STL
- added link arm_r5_link, mass 0.250000; collision cylinder length=0.1 radius=0.04; visual mesh filename=../meshes/arm_r5_link.STL
- added link arm_r6_link, mass 0.600000; visual mesh filename=../meshes/arm_r6_link.STL
- added link head_yaw_link, mass 0.496681; collision box size=0.1 0.2 0.2; visual mesh filename=../meshes/head_yaw_link.STL
- added link l_foot_heel
- added link l_foot_toe
- added link r_foot_heel
- added link r_foot_toe
- added link waist_yaw_link, mass 8.000000; collision box size=0.2 0.39 0.1; visual mesh filename=../meshes/waist_yaw_link.STL
- link base_link: mass 31.110854 -> 11.000; geometry collision box size=0.2 0.3 0.3; visual mesh filename=../meshes/base_link.STL
- link leg_l1_link: mass 1.703116 -> 1.900000; geometry visual mesh filename=../meshes/leg_l1_link.STL
- link leg_l2_link: mass 1.099494 -> 1.529802; geometry collision cylinder length=0.24 radius=0.08; visual mesh filename=../meshes/leg_l2_link.STL
- link leg_l3_link: mass 11.2873798308346 -> 10.000000; geometry collision box size=0.1 0.2 0.1; visual mesh filename=../meshes/leg_l3_link.STL
- link leg_l4_link: mass 3.235545 -> 2.600000; geometry collision box size=0.1 0.28 0.08; collision cylinder length=0.09 radius=0.04
- link leg_l5_link: mass 0.179272166113496 -> 0.050922; geometry visual mesh filename=../meshes/leg_l5_link.STL
- link leg_l6_link: mass 0.359578868782819 -> 0.365700; geometry collision box size=0.1 0.01 0.2; visual mesh filename=../meshes/leg_l6_link.STL
- link leg_r1_link: mass 0.812038227652222 -> 1.900000; geometry visual mesh filename=../meshes/leg_r1_link.STL
- link leg_r2_link: mass 1.09949380454122 -> 1.529802; geometry collision cylinder length=0.24 radius=0.08; visual mesh filename=../meshes/leg_r2_link.STL
- link leg_r3_link: mass 11.2704290325054 -> 10.000000; geometry collision box size=0.1 0.2 0.1; visual mesh filename=../meshes/leg_r3_link.STL
- link leg_r4_link: mass 1.6873629685696 -> 2.600000; geometry collision box size=0.1 0.28 0.08; collision cylinder length=0.09 radius=0.04
- link leg_r5_link: mass 0.179272166113496 -> 0.050922; geometry visual mesh filename=../meshes/leg_r5_link.STL
- link leg_r6_link: mass 0.359578868782818 -> 0.373459; geometry collision box size=0.1 0.01 0.2; visual mesh filename=../meshes/leg_r6_link.STL
Joints:
- removed joint dummy
- added joint arm_l1_joint: type fixed, parent base_link, child arm_l1_link, origin xyz=0 0.095627 0.05921 rpy=1.8326 0 0, axis 0 0 1, limit lower=-3.1416 upper=3.1416 effort=36.0 velocity=12.0
- added joint arm_l2_joint: type fixed, parent arm_l1_link, child arm_l2_link, origin xyz=0.036 0 -0.0895 rpy=-1.5708 1.309 -1.5708, axis 0 0 1, limit lower=-0.4 upper=1.5708 effort=36.0 velocity=12.0
- added joint arm_l3_joint: type fixed, parent arm_l2_link, child arm_l3_link, origin xyz=0.064778 -0.087206 -0.036 rpy=-1.8326 1.5708 0, axis 0 0 -1, limit lower=-2.0 upper=2.0 effort=36.0 velocity=12.0
- added joint arm_l4_joint: type fixed, parent arm_l3_link, child arm_l4_link, origin xyz=0.028 0 -0.1785 rpy=1.5708 0 1.5708, axis 0 0 -1, limit lower=-2.4 upper=0.0 effort=36.0 velocity=12.0
- added joint arm_l5_joint: type fixed, parent arm_l4_link, child arm_l5_link, origin xyz=0 -0.0835 -0.028 rpy=1.5708 1.5708 0, axis 0 0 1, limit lower=-2.0 upper=2.0 effort=9.0 velocity=12.0
- added joint arm_l6_joint: type fixed, parent arm_l5_link, child arm_l6_link, origin xyz=0.0245 0 0.0975 rpy=0 1.5708 0, axis 0 0 -1, limit lower=-1.5708 upper=1.5708 effort=9.0 velocity=12.0
- added joint arm_r1_joint: type fixed, parent base_link, child arm_r1_link, origin xyz=0 -0.095623 0.05921 rpy=1.309 0 0, axis 0 0 -1, limit lower=-3.1416 upper=3.1416 effort=36.0 velocity=12.0
- added joint arm_r2_joint: type fixed, parent arm_r1_link, child arm_r2_link, origin xyz=0.036 0 0.0895 rpy=1.5708 1.309 1.5708, axis 0 0 1, limit lower=-1.5708 upper=0.4 effort=36.0 velocity=12.0
- added joint arm_r3_joint: type fixed, parent arm_r2_link, child arm_r3_link, origin xyz=-0.064778 -0.087206 -0.036 rpy=-1.309 1.5708 0, axis 0 0 -1, limit lower=-2.0 upper=2.0 effort=36.0 velocity=12.0
- added joint arm_r4_joint: type fixed, parent arm_r3_link, child arm_r4_link, origin xyz=0.028 0 -0.1785 rpy=1.5708 0 1.5708, axis 0 0 1, limit lower=-2.4 upper=0.0 effort=36.0 velocity=12.0
- added joint arm_r5_joint: type fixed, parent arm_r4_link, child arm_r5_link, origin xyz=0 -0.0835 -0.028 rpy=1.5708 1.5708 0, axis 0 0 1, limit lower=-2.0 upper=2.0 effort=9.0 velocity=12.0
- added joint arm_r6_joint: type fixed, parent arm_r5_link, child arm_r6_link, origin xyz=0.0245 0 0.0975 rpy=0 1.5708 0, axis 0 0 -1, limit lower=-1.5708 upper=1.5708 effort=9.0 velocity=12.0
- added joint dummy_to_base_link: type continuous, parent dummy_link, child base_link, origin xyz=0 0 0 rpy=0 0 0
- added joint head_yaw_joint: type fixed, parent base_link, child head_yaw_link, origin xyz=0 0 0.1395 rpy=0 0 0, axis 0 0 -1, limit lower=-1.5708 upper=1.5708 effort=9.0 velocity=12.0
- added joint l_foot_heel_joint: type fixed, parent leg_l6_link, child l_foot_heel, origin xyz=0 -0.033 -0.0445 rpy=0 0 0
- added joint l_foot_toe_joint: type fixed, parent leg_l6_link, child l_foot_toe, origin xyz=0 -0.033 0.1415 rpy=0 0 0
- added joint r_foot_heel_joint: type fixed, parent leg_r6_link, child r_foot_heel, origin xyz=0 -0.033 -0.0445 rpy=0 0 0
- added joint r_foot_toe_joint: type fixed, parent leg_r6_link, child r_foot_toe, origin xyz=0 -0.033 0.1415 rpy=0 0 0
- added joint waist_yaw_joint: type fixed, parent base_link, child waist_yaw_link, origin xyz=0 0 -0.24015 rpy=0 0 0, axis 0 0 1, limit lower=-1.5708 upper=1.5708 effort=150.0 velocity=12.0
- joint leg_l1_joint: axis -1 0 0 -> 0 0 1; limit (none) -> lower=-0.2 upper=1.5708 effort=150.0 velocity=12.0; origin xyz=0.016745166004061 0.158 -0.0250735931288075 rpy=0 0.785398163397454 3.14159265358979 -> xyz=-0.0718 0.14977 -0.12986 rpy=0 1.5708 0; parent base_link -> waist_yaw_link; type continuous -> revolute
- joint leg_l2_joint: axis -1 0 0 -> 0 0 -1; limit (none) -> lower=-1.5708 upper=1.5708 effort=90.0 velocity=12.0; origin xyz=0.0800000000000011 0 -0.0420000000000002 rpy=0.585706330182336 1.57079631189374 -2.51846950759238 -> xyz=-0.028 0 0.0718 rpy=0 -1.5708 0; type continuous -> revolute
- joint leg_l3_joint: axis 0 -1 0 -> 0 0 1; limit (none) -> lower=-1.5708 upper=1.5708 effort=320.0 velocity=12.0; origin xyz=0.092 0 -0.08 rpy=0 -0.785398163397442 0 -> xyz=0 0.0823 -0.165 rpy=1.5708 0 0; type continuous -> revolute
- joint leg_l4_joint: axis 0 -1 0 -> 0 0 -1; limit (none) -> lower=0.0 upper=2.356 effort=320.0 velocity=12.0; origin xyz=0 0 -0.459104968164964 rpy=0 0 0 -> xyz=0 -0.38 0.0748 rpy=0 0 0; type continuous -> revolute
- joint leg_l5_joint: axis 0 1 0 -> 0 0 1; limit (none) -> lower=-0.8 upper=0.8 effort=70.0 velocity=12.0; origin xyz=2.21008500064235E-05 0 -0.321306622119717 rpy=0 0 0 -> xyz=0.0098491 -0.37124 0.0035 rpy=0 0 0; type continuous -> revolute
- joint leg_l6_joint: axis 0.99999999763436 0 6.87842964705043E-05 -> 0 0 1; limit (none) -> lower=-0.5236 upper=0.5236 effort=70.0 velocity=12.0; origin xyz=0 0 0 rpy=0 0 0 -> xyz=-0.011 0 0.011 rpy=0 1.5708 0; type continuous -> revolute
- joint leg_r1_joint: axis -1 0 0 -> 0 0 1; limit (none) -> lower=-1.5708 upper=0.2 effort=150.0 velocity=12.0; origin xyz=0.0167451660040608 -0.158 -0.0250735931288074 rpy=0 0.785398163397455 3.14159265358979 -> xyz=-0.0718 -0.14977 -0.12986 rpy=0 1.5708 0; parent base_link -> waist_yaw_link; type continuous -> revolute
- joint leg_r2_joint: axis -1 0 0 -> 0 0 -1; limit (none) -> lower=-1.5708 upper=1.5708 effort=90.0 velocity=12.0; origin xyz=0.0800000000000007 0 -0.0419999999999999 rpy=3.14159265358979 1.5707963267949 0 -> xyz=-0.028 0 0.0718 rpy=0 -1.5708 0; type continuous -> revolute
- joint leg_r3_joint: axis 0 -1 0 -> 0 0 1; limit (none) -> lower=-1.5708 upper=1.5708 effort=320.0 velocity=12.0; origin xyz=0.0920000000000001 0 -0.08 rpy=0 -0.785398163397442 0 -> xyz=0 0.0823 -0.165 rpy=1.5708 0 0; type continuous -> revolute
- joint leg_r4_joint: axis 0 -1 0 -> 0 0 -1; limit (none) -> lower=0.0 upper=2.356 effort=320.0 velocity=12.0; origin xyz=0 0 -0.459104968164964 rpy=0 0 0 -> xyz=0 -0.38 0.0748 rpy=0 0 0; type continuous -> revolute
- joint leg_r5_joint: axis 0 1 0 -> 0 0 1; limit (none) -> lower=-0.8 upper=0.8 effort=70.0 velocity=12.0; origin xyz=2.21008500065345E-05 0 -0.321306622119717 rpy=0 0 0 -> xyz=0.0098491 -0.37124 0.0035 rpy=0 0 0; type continuous -> revolute
- joint leg_r6_joint: axis 0.99999999763436 0 6.87842964705043E-05 -> 0 0 1; limit (none) -> lower=-0.5236 upper=0.5236 effort=70.0 velocity=12.0; origin xyz=0 0 0 rpy=0 0 0 -> xyz=-0.011 0 0.011 rpy=0 1.5708 0; type continuous -> revolute

File: humanoid-legged-description/urdf/humanoid_legged_control.urdf (robot description, URDF)
Before this commit: robot humanoid_legged_description, 20 links, 19 joints
Links:
- removed link l_foot_side
- removed link r_foot_side
- added link arm_l1_link, mass 0.565198
- added link arm_l2_link, mass 0.850000
- added link arm_l3_link, mass 0.700000; collision cylinder length=0.16 radius=0.04
- added link arm_l4_link, mass 0.443929
- added link arm_l5_link, mass 0.250000; collision cylinder length=0.1 radius=0.04
- added link arm_l6_link, mass 0.600000
- added link arm_r1_link, mass 0.565198
- added link arm_r2_link, mass 0.850000
- added link arm_r3_link, mass 0.700000; collision cylinder length=0.16 radius=0.04
- added link arm_r4_link, mass 0.443929
- added link arm_r5_link, mass 0.250000; collision cylinder length=0.1 radius=0.04
- added link arm_r6_link, mass 0.600000
- added link head_yaw_link, mass 0.496681; collision box size=0.1 0.2 0.2
- added link waist_yaw_link, mass 8.000000; collision box size=0.2 0.39 0.1
- link base_link: mass 31.110854 -> 11.000; geometry collision box size=0.2 0.3 0.3
- link l_foot_toe: geometry 
- link leg_l1_link: mass 1.703116 -> 1.900000
- link leg_l2_link: mass 1.099494 -> 1.529802; geometry collision cylinder length=0.24 radius=0.08
- link leg_l3_link: mass 11.2873798308346 -> 10.000000; geometry collision box size=0.1 0.2 0.1
- link leg_l4_link: mass 3.235545 -> 2.600000; geometry collision box size=0.1 0.28 0.08; collision cylinder length=0.09 radius=0.04
- link leg_l5_link: mass 0.179272166113496 -> 0.050922
- link leg_l6_link: mass 0.359578868782819 -> 0.365700; geometry collision box size=0.1 0.01 0.2
- link leg_r1_link: mass 0.812038227652222 -> 1.900000
- link leg_r2_link: mass 1.09949380454122 -> 1.529802; geometry collision cylinder length=0.24 radius=0.08
- link leg_r3_link: mass 11.2704290325054 -> 10.000000; geometry collision box size=0.1 0.2 0.1
- link leg_r4_link: mass 1.6873629685696 -> 2.600000; geometry collision box size=0.1 0.28 0.08; collision cylinder length=0.09 radius=0.04
- link leg_r5_link: mass 0.179272166113496 -> 0.050922
- link leg_r6_link: mass 0.359578868782818 -> 0.373459; geometry collision box size=0.1 0.01 0.2
- link r_foot_heel: geometry 
- link r_foot_toe: geometry 
Joints:
- removed joint l_foot_side_joint
- removed joint r_foot_side_joint
- added joint arm_l1_joint: type fixed, parent base_link, child arm_l1_link, origin xyz=0 0.095627 0.05921 rpy=1.8326 0 0, axis 0 0 1, limit lower=-3.1416 upper=3.1416 effort=36.0 velocity=12.0
- added joint arm_l2_joint: type fixed, parent arm_l1_link, child arm_l2_link, origin xyz=0.036 0 -0.0895 rpy=-1.5708 1.309 -1.5708, axis 0 0 1, limit lower=-0.4 upper=1.5708 effort=36.0 velocity=12.0
- added joint arm_l3_joint: type fixed, parent arm_l2_link, child arm_l3_link, origin xyz=0.064778 -0.087206 -0.036 rpy=-1.8326 1.5708 0, axis 0 0 -1, limit lower=-2.0 upper=2.0 effort=36.0 velocity=12.0
- added joint arm_l4_joint: type fixed, parent arm_l3_link, child arm_l4_link, origin xyz=0.028 0 -0.1785 rpy=1.5708 0 1.5708, axis 0 0 -1, limit lower=-2.4 upper=0.0 effort=36.0 velocity=12.0
- added joint arm_l5_joint: type fixed, parent arm_l4_link, child arm_l5_link, origin xyz=0 -0.0835 -0.028 rpy=1.5708 1.5708 0, axis 0 0 1, limit lower=-2.0 upper=2.0 effort=9.0 velocity=12.0
- added joint arm_l6_joint: type fixed, parent arm_l5_link, child arm_l6_link, origin xyz=0.0245 0 0.0975 rpy=0 1.5708 0, axis 0 0 -1, limit lower=-1.5708 upper=1.5708 effort=9.0 velocity=12.0
- added joint arm_r1_joint: type fixed, parent base_link, child arm_r1_link, origin xyz=0 -0.095623 0.05921 rpy=1.309 0 0, axis 0 0 -1, limit lower=-3.1416 upper=3.1416 effort=36.0 velocity=12.0
- added joint arm_r2_joint: type fixed, parent arm_r1_link, child arm_r2_link, origin xyz=0.036 0 0.0895 rpy=1.5708 1.309 1.5708, axis 0 0 1, limit lower=-1.5708 upper=0.4 effort=36.0 velocity=12.0
- added joint arm_r3_joint: type fixed, parent arm_r2_link, child arm_r3_link, origin xyz=-0.064778 -0.087206 -0.036 rpy=-1.309 1.5708 0, axis 0 0 -1, limit lower=-2.0 upper=2.0 effort=36.0 velocity=12.0
- added joint arm_r4_joint: type fixed, parent arm_r3_link, child arm_r4_link, origin xyz=0.028 0 -0.1785 rpy=1.5708 0 1.5708, axis 0 0 1, limit lower=-2.4 upper=0.0 effort=36.0 velocity=12.0
- added joint arm_r5_joint: type fixed, parent arm_r4_link, child arm_r5_link, origin xyz=0 -0.0835 -0.028 rpy=1.5708 1.5708 0, axis 0 0 1, limit lower=-2.0 upper=2.0 effort=9.0 velocity=12.0
- added joint arm_r6_joint: type fixed, parent arm_r5_link, child arm_r6_link, origin xyz=0.0245 0 0.0975 rpy=0 1.5708 0, axis 0 0 -1, limit lower=-1.5708 upper=1.5708 effort=9.0 velocity=12.0
- added joint head_yaw_joint: type fixed, parent base_link, child head_yaw_link, origin xyz=0 0 0.1395 rpy=0 0 0, axis 0 0 -1, limit lower=-1.5708 upper=1.5708 effort=9.0 velocity=12.0
- added joint waist_yaw_joint: type fixed, parent base_link, child waist_yaw_link, origin xyz=0 0 -0.24015 rpy=0 0 0, axis 0 0 1, limit lower=-1.5708 upper=1.5708 effort=150.0 velocity=12.0
- joint l_foot_heel_joint: origin xyz=-0.0445 0 -0.038 rpy=0 0 0 -> xyz=0 -0.033 -0.0445 rpy=0 0 0
- joint l_foot_toe_joint: origin xyz=0.1415 0 -0.038 rpy=0 0 0 -> xyz=0 -0.033 0.1415 rpy=0 0 0
- joint leg_l1_joint: axis -1 0 0 -> 0 0 1; limit lower=-1.57 upper=1.57 effort=150.0 velocity=7.5 -> lower=-0.2 upper=1.5708 effort=150.0 velocity=12.0; origin xyz=0.016745166004061 0.158 -0.0250735931288075 rpy=0 0.785398163397454 3.14159265358979 -> xyz=-0.0718 0.14977 -0.12986 rpy=0 1.5708 0; parent base_link -> waist_yaw_link
- joint leg_l2_joint: axis -1 0 0 -> 0 0 -1; limit lower=-1.57 upper=1.57 effort=150.0 velocity=7.5 -> lower=-1.5708 upper=1.5708 effort=90.0 velocity=12.0; origin xyz=0.0800000000000011 0 -0.0420000000000002 rpy=0.585706330182336 1.57079631189374 -2.51846950759238 -> xyz=-0.028 0 0.0718 rpy=0 -1.5708 0
- joint leg_l3_joint: axis 0 -1 0 -> 0 0 1; limit lower=-0.90 upper=1.57 effort=300.0 velocity=7.5 -> lower=-1.5708 upper=1.5708 effort=320.0 velocity=12.0; origin xyz=0.092 0 -0.08 rpy=0 -0.785398163397442 0 -> xyz=0 0.0823 -0.165 rpy=1.5708 0 0
- joint leg_l4_joint: axis 0 -1 0 -> 0 0 -1; limit lower=-1.7 upper=0.1 effort=300.0 velocity=7.5 -> lower=0.0 upper=2.356 effort=320.0 velocity=12.0; origin xyz=0 0 -0.459104968164964 rpy=0 0 0 -> xyz=0 -0.38 0.0748 rpy=0 0 0
- joint leg_l5_joint: axis 0 1 0 -> 0 0 1; limit lower=-1.0 upper=1.0 effort=90.0 velocity=7.5 -> lower=-0.8 upper=0.8 effort=70.0 velocity=12.0; origin xyz=2.21008500064235E-05 0 -0.321306622119717 rpy=0 0 0 -> xyz=0.0098491 -0.37124 0.0035 rpy=0 0 0
- joint leg_l6_joint: axis 0.99999999763436 0 6.87842964705043E-05 -> 0 0 1; limit lower=-1.0 upper=1.0 effort=90.0 velocity=7.5 -> lower=-0.5236 upper=0.5236 effort=70.0 velocity=12.0; origin xyz=0 0 0 rpy=0 0 0 -> xyz=-0.011 0 0.011 rpy=0 1.5708 0
- joint leg_r1_joint: axis -1 0 0 -> 0 0 1; limit lower=-1.57 upper=1.57 effort=150.0 velocity=7.5 -> lower=-1.5708 upper=0.2 effort=150.0 velocity=12.0; origin xyz=0.0167451660040608 -0.158 -0.0250735931288074 rpy=0 0.785398163397455 3.14159265358979 -> xyz=-0.0718 -0.14977 -0.12986 rpy=0 1.5708 0; parent base_link -> waist_yaw_link
- joint leg_r2_joint: axis -1 0 0 -> 0 0 -1; limit lower=-1.57 upper=1.57 effort=150.0 velocity=7.5 -> lower=-1.5708 upper=1.5708 effort=90.0 velocity=12.0; origin xyz=0.0800000000000007 0 -0.0419999999999999 rpy=3.14159265358979 1.5707963267949 0 -> xyz=-0.028 0 0.0718 rpy=0 -1.5708 0
- joint leg_r3_joint: axis 0 -1 0 -> 0 0 1; limit lower=-0.90 upper=1.57 effort=300.0 velocity=7.5 -> lower=-1.5708 upper=1.5708 effort=320.0 velocity=12.0; origin xyz=0.0920000000000001 0 -0.08 rpy=0 -0.785398163397442 0 -> xyz=0 0.0823 -0.165 rpy=1.5708 0 0
- joint leg_r4_joint: axis 0 -1 0 -> 0 0 -1; limit lower=-1.7 upper=0.1 effort=300.0 velocity=7.5 -> lower=0.0 upper=2.356 effort=320.0 velocity=12.0; origin xyz=0 0 -0.459104968164964 rpy=0 0 0 -> xyz=0 -0.38 0.0748 rpy=0 0 0
- joint leg_r5_joint: axis 0 1 0 -> 0 0 1; limit lower=-1.0 upper=1.0 effort=90.0 velocity=7.5 -> lower=-0.8 upper=0.8 effort=70.0 velocity=12.0; origin xyz=2.21008500065345E-05 0 -0.321306622119717 rpy=0 0 0 -> xyz=0.0098491 -0.37124 0.0035 rpy=0 0 0
- joint leg_r6_joint: axis 0.99999999763436 0 6.87842964705043E-05 -> 0 0 1; limit lower=-1.0 upper=1.0 effort=90.0 velocity=7.5 -> lower=-0.5236 upper=0.5236 effort=70.0 velocity=12.0; origin xyz=0 0 0 rpy=0 0 0 -> xyz=-0.011 0 0.011 rpy=0 1.5708 0
- joint r_foot_heel_joint: origin xyz=-0.0445 0 -0.038 rpy=0 0 0 -> xyz=0 -0.033 -0.0445 rpy=0 0 0
- joint r_foot_toe_joint: origin xyz=0.1415 0 -0.038 rpy=0 0 0 -> xyz=0 -0.033 0.1415 rpy=0 0 0
